Commit message: tqdm for loop while colleting data

File: xacros/debur_with_full_tactile.urdf.xacro (robot description, xacro)
@@ -8,5 +8,5 @@
         <parent link="TCP"/>
         <child link="davis"/>
-	    <origin xyz="-0.084363 0.07636588 0.11668644" rpy="-1.6191409 0.0151598 0.0068846"/>
+	    <origin xyz="0.07 0.09 0.13" rpy="-1.5708 0 -1.5708"/>
     </joint>
     <joint name="TCP_to_pressure_ft" type="fixed">
