Commit message: make generic files to avoid accidents

File: xacros/sample_tool.urdf.xacro (robot description, xacro)
@@ -7,5 +7,5 @@
         <parent link="TCP"/>
         <child link="davis"/>
-	    <origin xyz="-0.10126922 0.07627988 0.11786909" rpy="-1.56978981 -0.02018286 0.04749861"/>
+	    <origin xyz="x y z" rpy="r p y"/>
     </joint>
     <joint name="TCP_to_pressure_ft" type="fixed">
